File: pcb/arch_40.kicad_pcb (KiCad board)
At the start: 2 copper layers, 100 parts, among them SW0-1 SWITCH_PUSH, SW0-2 SWITCH_PUSH, SW0-3 SWITCH_PUSH, SW0-4 SWITCH_PUSH, SW1-1 SWITCH_PUSH, SW1-2 SWITCH_PUSH, SW1-3 SWITCH_PUSH, SW10-1 SWITCH_PUSH, SW10-2 SWITCH_PUSH, SW10-3 SWITCH_PUSH, SW10-4 SWITCH_PUSH, SW11-1 SWITCH_PUSH, SW11-2 SWITCH_PUSH, SW11-3 SWITCH_PUSH, SW12-1 SWITCH_PUSH, SW12-2 SWITCH_PUSH, SW12-3 SWITCH_PUSH, SW12-4 SWITCH_PUSH, SW2-1 SWITCH_PUSH, SW2-2 SWITCH_PUSH, SW2-3 SWITCH_PUSH, SW2-4 SWITCH_PUSH, SW3-1 SWITCH_PUSH, SW3-2 SWITCH_PUSH, SW3-3 SWITCH_PUSH, SW3-4 SWITCH_PUSH, SW4-1 SWITCH_PUSH, SW4-2 SWITCH_PUSH, SW4-3 SWITCH_PUSH, SW4-4 SWITCH_PUSH, SW5-1 SWITCH_PUSH, SW5-2 SWITCH_PUSH, SW5-3 SWITCH_PUSH, SW5-4 SWITCH_PUSH, SW6-1 SWITCH_PUSH, SW6-2 SWITCH_PUSH, SW6-3 SWITCH_PUSH, SW7-1 SWITCH_PUSH, SW7-2 SWITCH_PUSH, SW7-3 SWITCH_PUSH, SW7-4 SWITCH_PUSH, SW8-1 SWITCH_PUSH, SW8-2 SWITCH_PUSH, SW8-3 SWITCH_PUSH, SW8-4 SWITCH_PUSH, SW9-1 SWITCH_PUSH, SW9-2 SWITCH_PUSH, SW9-3 SWITCH_PUSH, SW9-4 SWITCH_PUSH, U1 ARDUINO_PRO_MICRO

Commit message: pcb. placed the footprints accordingly.
Parts:
- U1: moved to B.Cu
- moved U1 133.8 mm to (148.7, 105.3)
- moved SW-RST1 127.1 mm to (136.7, 98.0)
- moved SW0-1 52.7 mm to (35.1, 42.2), turned to 165 degrees
- moved D0-1 49.5 mm to (31.9, 50.1), turned to 165 degrees
- moved SW0-2 47.7 mm to (30.1, 60.6), turned to 165 degrees
- moved D0-2 45.1 mm to (27.5, 68.7), turned to 165 degrees
- moved SW0-3 42.8 mm to (25.2, 79.0), turned to 165 degrees
- moved D0-3 40.4 mm to (22.8, 86.9), turned to 165 degrees
- moved D5-4 39.1 mm to (115.6, 126.8), turned to 165 degrees
- moved SW5-4 38.3 mm to (118.2, 118.8), turned to 165 degrees
- moved D6-2 38.3 mm to (155.2, 149.6), turned to 340 degrees
- moved SW0-4 37.8 mm to (20.3, 97.4), turned to 165 degrees
- moved SW5-3 36.7 mm to (123.0, 100.3), turned to 165 degrees
- moved D5-3 36.7 mm to (121.0, 108.3), turned to 165 degrees
- moved D7-4 36.3 mm to (179.4, 126.3), turned to 195 degrees
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