File: pcb/arch_40.kicad_pcb (KiCad board)
At the start: 2 copper layers, 275.5 x 130.3 mm, 100 parts, among them SW0-1 SWITCH_PUSH, SW0-2 SWITCH_PUSH, SW0-3 SWITCH_PUSH, SW0-4 SWITCH_PUSH, SW1-1 SWITCH_PUSH, SW1-2 SWITCH_PUSH, SW1-3 SWITCH_PUSH, SW10-1 SWITCH_PUSH, SW10-2 SWITCH_PUSH, SW10-3 SWITCH_PUSH, SW10-4 SWITCH_PUSH, SW11-1 SWITCH_PUSH, SW11-2 SWITCH_PUSH, SW11-3 SWITCH_PUSH, SW12-1 SWITCH_PUSH, SW12-2 SWITCH_PUSH, SW12-3 SWITCH_PUSH, SW12-4 SWITCH_PUSH, SW2-1 SWITCH_PUSH, SW2-2 SWITCH_PUSH, SW2-3 SWITCH_PUSH, SW2-4 SWITCH_PUSH, SW3-1 SWITCH_PUSH, SW3-2 SWITCH_PUSH, SW3-3 SWITCH_PUSH, SW3-4 SWITCH_PUSH, SW4-1 SWITCH_PUSH, SW4-2 SWITCH_PUSH, SW4-3 SWITCH_PUSH, SW4-4 SWITCH_PUSH, SW5-1 SWITCH_PUSH, SW5-2 SWITCH_PUSH, SW5-3 SWITCH_PUSH, SW5-4 SWITCH_PUSH, SW6-1 SWITCH_PUSH, SW6-2 SWITCH_PUSH, SW6-3 SWITCH_PUSH, SW7-1 SWITCH_PUSH, SW7-2 SWITCH_PUSH, SW7-3 SWITCH_PUSH, SW7-4 SWITCH_PUSH, SW8-1 SWITCH_PUSH, SW8-2 SWITCH_PUSH, SW8-3 SWITCH_PUSH, SW8-4 SWITCH_PUSH, SW9-1 SWITCH_PUSH, SW9-2 SWITCH_PUSH, SW9-3 SWITCH_PUSH, SW9-4 SWITCH_PUSH, U1 ARDUINO_PRO_MICRO

Commit message: added holes to match the cutout.
Parts:
- added ?: MountingHole_4.3mm_M4_ISO7380, MountingHole:MountingHole_4.3mm_M4_ISO7380, F.Cu at (162.2, 113.9)
- added ?: MountingHole_4.3mm_M4_ISO7380, MountingHole:MountingHole_4.3mm_M4_ISO7380, F.Cu at (133.0, 114.2)
- added ?: MountingHole_4.3mm_M4_ISO7380, MountingHole:MountingHole_4.3mm_M4_ISO7380, F.Cu at (153.2, 76.8)
- added ?: MountingHole_4.3mm_M4_ISO7380, MountingHole:MountingHole_4.3mm_M4_ISO7380, F.Cu at (142.2, 77.1)
- moved SW9-1 0.20 mm to (196.9, 44.2)
- moved SW8-4 0.17 mm to (194.6, 108.8)
Routing:
- net /ROW-3: track 406.8 -> 407.7 mm
- net /COL8: track 136.9 -> 137.6 mm
- net /COL12: track 214.5 -> 213.9 mm
